File: hardware/Sensor-Boi.kicad_pcb (KiCad board)
At the start: 2 copper layers, 152 x 86.8 mm, 29 parts, among them Q1 2N7002, U1 ESP32-S3-WROOM-1, U10 CP2102N-A02-GQFN24R, U2 MAX31856, U3 SN65HVD230, U4 LM2596S-5, U5 AMS1117-3.3, U6 6N137, U7 ISO7741DWR, U8 LTC4412ES6_TRPBF, U9 B0505LS-1WR3_C7465180

Commit message: complete power subsystem
Parts:
- added C5: 47uF 16V, Capacitor_SMD:CP_Elec_5x5.4, F.Cu at (110.4, 55.8)
- added C6: 100nF, PCM_JLCPCB:C_0402, F.Cu at (114.6, 45.5)
- added C7: 100uF 50V, Capacitor_SMD:CP_Elec_6.3x7.7, F.Cu at (100.7, 56.4)
- added D2: SS34, PCM_JLCPCB:D_SMA, F.Cu at (110.0, 61.5)
- added D6: PRTR5V0U2X, Package_TO_SOT_SMD:SOT-143, F.Cu at (115.3, 42.4)
- added R10: 100Ω, PCM_JLCPCB:R_0402, F.Cu at (114.6, 47.4)
- added U11: LM2596S-3.3, Package_TO_SOT_SMD:TO-263-5_TabPin3, F.Cu at (106.2, 46.2)
