File: hardware/Sensor-Boi.kicad_sch (KiCad schematic)
At the start: 31 parts, among them Q1 2N7002, U1 ESP32-S3-WROOM-1, U2 MAX31856, U3 SN65HVD230, U4 LM2596S-5, U5 AMS1117-3.3, U6 6N137, U7 ISO7741DWR, U8 LTC4412ES6_TRPBF, U9 B0505LS-1WR3_C7465180

Commit message: complete power subsystem
Parts:
- removed C5: 22uF, PCM_JLCPCB:C_1206, symbol PCM_JLCPCB-Capacitors:1206,22uF
- removed D2: SMBJ15A, PCM_JLCPCB:D_SMB, symbol PCM_JLCPCB-Diodes:TVS-Uni,SMBJ15A
- removed D5: BZX84C5V1, PCM_JLCPCB:D_SOT-23, symbol PCM_JLCPCB-Diodes:Zener,BZX84C5V1
- removed L1: 22uH,5mA, PCM_JLCPCB:L_0805, symbol PCM_JLCPCB-Inductors:22uH,5mA
- removed U4: LM2596S-5, Package_TO_SOT_SMD:TO-263-5_TabPin3, symbol Regulator_Switching:LM2596S-5
- removed U5: AMS1117-3.3, Package_TO_SOT_SMD:SOT-223-3_TabPin2, symbol Regulator_Linear:AMS1117-3.3
- added C5: 47uF 16V, Capacitor_SMD:CP_Elec_5x5.4, symbol Device:C_Polarized
- added C6: 100nF, PCM_JLCPCB:C_0402, symbol PCM_JLCPCB-Capacitors:0402,100nF
- added C7: 100uF 50V, Capacitor_SMD:CP_Elec_6.3x7.7, symbol Device:C_Polarized
- added D2: SS34, PCM_JLCPCB:D_SMA, symbol PCM_JLCPCB-Diodes:Schottky,SS34
- added D6: PRTR5V0U2X, Package_TO_SOT_SMD:SOT-143, symbol Power_Protection:PRTR5V0U2X
- added L1: 22uH, Inductor_SMD:L_4.0x4.0mm_Pad2.0x2.4mm, symbol Device:L
- added R10: 100Ω, PCM_JLCPCB:R_0402, symbol PCM_JLCPCB-Resistors:0402,100kΩ
- added U10: 74LVC1G14, symbol 74xGxx:74LVC1G14
- added U11: LM2596S-3.3, Package_TO_SOT_SMD:TO-263-5_TabPin3, symbol Regulator_Switching:LM2596S-3.3
Connections:
- net 12V: now also C7.1, U11.1 (VIN)
- net 3V3: now also C5.1, D6.4 (VCC), L1.2, U10.5 (VCC), U11.4 (FB)
- net GND: now also C5.2, C7.2, D2.1, D6.1 (GND), U10.3 (GND), U11.3 (GND), U11.5 (~{ON}/OFF)
- net Wheel_Speed_MCU: now also U10.4
- new net: D2.2, L1.1, U11.2 (OUT)
- new net: D6.2 (I/O1), R10.2
- new net Hall_Sensor: C6.1, R10.1
Other:
- note added: "Wheel Speed"
